File: pcb/Split_Rail_Supply/Split_Rail_Supply.kicad_pcb (KiCad board)
At the start: 2 copper layers, 17 parts, among them J1 Header_01x02_Wurth_61300211121, U1 TPS563206

Commit message: Update SCH, PCB
Parts:
- removed J1: Header_01x02_Wurth_61300211121, Connector_PinHeader_2.54mm:PinHeader_1x02_P2.54mm_Vertical
- added C11: 10uF,25V,X5R,0603, Capacitor_SMD:C_0603_1608Metric_Pad1.08x0.95mm_HandSolder, F.Cu at (138.4, 103.6)
- added D2: 150060GS75000, LED_SMD:LED_0603_1608Metric_Pad1.05x0.95mm_HandSolder, F.Cu at (132.7, 96.8)
- added D3: 150060GS75000, LED_SMD:LED_0603_1608Metric_Pad1.05x0.95mm_HandSolder, F.Cu at (157.8, 83.2)
- added D4: 150060GS75000, LED_SMD:LED_0603_1608Metric_Pad1.05x0.95mm_HandSolder, F.Cu at (137.4, 83.4)
- added H1: MountingHole, MountingHole:MountingHole_2.7mm_M2.5_DIN965, F.Cu at (131.0, 83.0)
- added H2: MountingHole, MountingHole:MountingHole_2.7mm_M2.5_DIN965, F.Cu at (163.0, 83.0)
- added H3: MountingHole, MountingHole:MountingHole_2.7mm_M2.5_DIN965, F.Cu at (163.0, 110.0)
- added H4: MountingHole, MountingHole:MountingHole_2.7mm_M2.5_DIN965, F.Cu at (131.0, 110.0)
- added J2: Header_01x02_Wurth_61300211121, Connector_PinHeader_2.54mm:PinHeader_1x02_P2.54mm_Vertical, F.Cu at (153.7, 89.5)
- added J4: JST_B2B-PH-K-x, Connector_JST:JST_PH_B2B-PH-K_1x02_P2.00mm_Vertical, F.Cu at (131.8, 102.8)
- added J5: JST_B2B-PH-K-x, Connector_JST:JST_PH_B2B-PH-K_1x02_P2.00mm_Vertical, F.Cu at (151.7, 84.0)
- added J6: JST_B2B-PH-K-x, Connector_JST:JST_PH_B2B-PH-K_1x02_P2.00mm_Vertical, F.Cu at (141.7, 83.8)
- added J7: Header_01x02_Wurth_61300211121, Connector_PinHeader_2.54mm:PinHeader_1x02_P2.54mm_Vertical, F.Cu at (142.1, 89.4)
- added J8: Header_01x02_Wurth_61300211121, Connector_PinHeader_2.54mm:PinHeader_1x02_P2.54mm_Vertical, F.Cu at (138.4, 109.3)
- added J9: JST_B2B-PH-K-x, Connector_JST:JST_PH_B2B-PH-K_1x02_P2.00mm_Vertical, F.Cu at (131.8, 93.0)
- added R4: 1k,0603, Resistor_SMD:R_0603_1608Metric_Pad0.98x0.95mm_HandSolder, F.Cu at (136.5, 94.8)
- added R5: 2k,0603, Resistor_SMD:R_0603_1608Metric_Pad0.98x0.95mm_HandSolder, F.Cu at (158.3, 88.9)
- added R6: 2k,0603, Resistor_SMD:R_0603_1608Metric_Pad0.98x0.95mm_HandSolder, F.Cu at (137.4, 87.0)
- C7: value 47uF,35V,Elec,6.6x6.6mm -> 10uF,25V,X5R,0603; footprint Capacitor_SMD:CP_Elec_6.3x7.7 -> Capacitor_SMD:C_0603_1608Metric_Pad1.08x0.95mm_HandSolder
- D1: value NSR0530HT1G -> DFLS230L-7; footprint Diode_SMD:D_SOD-323_HandSoldering -> Diode_SMD:D_PowerDI-123
- U1: value TPS563206 -> TPS564255
- moved D1 99.7 mm to (156.9, 103.2), turned to -90 degrees
- moved U1 99.5 mm to (143.5, 101.4)
- moved L1 96.5 mm to (150.0, 100.0)
- moved C10 92.8 mm to (160.5, 98.2), turned to 90 degrees
- moved C9 92.0 mm to (158.5, 98.2), turned to 90 degrees
- moved C8 91.3 mm to (156.5, 98.2), turned to 90 degrees
- moved C3 83.9 mm to (143.7, 97.1), turned to -90 degrees
- moved C7 81.9 mm to (136.9, 103.6), turned to 90 degrees
- moved C4 80.6 mm to (141.7, 97.1), turned to -90 degrees
- moved C5 77.3 mm to (139.7, 97.1), turned to -90 degrees
- moved C1 76.1 mm to (140.1, 102.3), turned to 90 degrees
- moved C2 75.9 mm to (141.6, 102.3), turned to 90 degrees
- moved R2 70.2 mm to (140.7, 99.8), turned to 180 degrees
- moved C6 69.8 mm to (137.8, 99.3), turned to -90 degrees
- moved R1 67.2 mm to (136.3, 99.3), turned to -90 degrees
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Connections:
- C6 pad 2: -Vout -> /FB
- L1 pad 1: Net-(U1-SW) -> GND
- L1 pad 2: GND -> Net-(U1-SW)
- L1 pad 3: GND -> Net-(D1-A)
- L1 pad 4: Net-(D1-A) -> GND
- R1 pad 2: -Vout -> /FB
- R2 pad 1: -Vout -> /FB
- U1 pad 6: -Vout -> /FB
Routing:
- net GND: track 0.00 -> 15.1 mm, vias 0 -> 4
- net -Vout: track 0.00 -> 14.8 mm
- net /FB: track 0.00 -> 7.90 mm
- net Net-(U1-SW): track 0.00 -> 5.24 mm
- net /Vin: track 0.00 -> 2.42 mm
- net Net-(J9-Pin_2): track 0.00 -> 1.05 mm, vias 0 -> 1
Other:
- board outline added: 38 x 33 mm

Commit message: Finalize RevA
Parts:
- J9: value JST_B2B-PH-K-x -> Header_01x02_Wurth_61300211121; footprint Connector_JST:JST_PH_B2B-PH-K_1x02_P2.00mm_Vertical -> Connector_PinHeader_2.54mm:PinHeader_1x02_P2.54mm_Vertical
- R1: value 10k,0603 -> 22k,0603
- R2: value 10k,0603 -> 3k,0603
- R3: value 0R,0603 -> 10k,0603
- moved J9 2.59 mm to (131.5, 90.4), turned to 0 degrees
- moved R5 2.04 mm to (157.9, 86.9)
- moved R4 1.92 mm to (134.8, 93.9)
- moved R3 1.73 mm to (134.8, 90.3)
- moved J7 0.83 mm to (141.4, 89.8)
- moved R2 0.61 mm to (140.1, 99.9), turned to 0 degrees
- moved J2 0.44 mm to (154.0, 89.8)
- moved D1 0.36 mm to (156.8, 102.8)
- moved C6 0.36 mm to (137.6, 99.0)
- moved R1 0.36 mm to (136.1, 99.0)
- moved J5 0.15 mm to (151.7, 83.8)
- moved D4 0.14 mm to (137.5, 83.3)
- moved D3 0.14 mm to (157.9, 83.3)
- moved R6 0.10 mm to (137.5, 87.0)
Connections:
- J9 pad 1: /Vin -> /En
- J9 pad 2: Net-(J9-Pin_2) -> -Vout
- R3 pad 2: Net-(J9-Pin_2) -> /En
- U1 pad 5: Net-(J9-Pin_2) -> /En
Routing:
- net -Vout: track 14.8 -> 57.1 mm
- net +Vout: track 0.00 -> 35.3 mm
- net GND: track 15.1 -> 49.7 mm, vias 4 -> 10
- net /Vin: track 2.42 -> 35.3 mm
- net /En: track 0.00 -> 24.2 mm, vias 0 -> 4
- net Net-(D1-A): track 0.00 -> 4.35 mm
- net Net-(D2-A): track 0.00 -> 3.10 mm
- net Net-(D4-A): track 0.00 -> 1.91 mm
- net Net-(D3-A): track 0.00 -> 1.81 mm
- net Net-(J9-Pin_2): track 1.05 -> 0.00 mm, vias 1 -> 0
- net /FB: track 7.90 -> 8.69 mm, vias 0 -> 2
- added copper zone on B.Cu, net GND
Other:
- board text added: "*"
- board text added: "+ -"
- board text added: "- +"
- board text added: "Disable"
- board text added: "Split Rail Supply Rev A"
- board text added: "Vin"
- board text added: "Vout+"
- board text added: "Vout-"
- board text added: "by fl0m0 2424-10-27"
