File: pcb/Split_Rail_Supply/Split_Rail_Supply.kicad_sch (KiCad schematic)
At the start: 17 parts, among them J1 Header_01x02_Wurth_61300211121, U1 TPS563206

Commit message: Update SCH, PCB
Parts:
- removed C7: 47uF,35V,Elec,6.6x6.6mm, Capacitor_SMD:CP_Elec_6.3x7.7, symbol Capacitor_User:47uF,35V,Elec,6.6x6.6mm
- removed J1: Header_01x02_Wurth_61300211121, Connector_PinHeader_2.54mm:PinHeader_1x02_P2.54mm_Vertical, symbol Connector_User:Pin_Header_01x02_Wurth_61300211121
- added C11, C7: 10uF,25V,X5R,0603, Capacitor_SMD:C_0603_1608Metric_Pad1.08x0.95mm_HandSolder, symbol Capacitor_User:10uF,25V,X5R,0603
- added D2, D3, D4: 150060GS75000, LED_SMD:LED_0603_1608Metric_Pad1.05x0.95mm_HandSolder, symbol LED_User:150060GS75000
- added H1, H2, H3, H4: MountingHole, MountingHole:MountingHole_2.7mm_M2.5_DIN965, symbol Mechanical:MountingHole
- added J2, J7, J8: Header_01x02_Wurth_61300211121, Connector_PinHeader_2.54mm:PinHeader_1x02_P2.54mm_Vertical, symbol Connector_User:Pin_Header_01x02_Wurth_61300211121
- added J4, J5, J6, J9: JST_B2B-PH-K-x, Connector_JST:JST_PH_B2B-PH-K_1x02_P2.00mm_Vertical, symbol Connector_User:JST_B2B-PH-K-x
- added R4: 1k,0603, Resistor_SMD:R_0603_1608Metric_Pad0.98x0.95mm_HandSolder, symbol Resistor_User:1k,0603
- added R5, R6: 2k,0603, Resistor_SMD:R_0603_1608Metric_Pad0.98x0.95mm_HandSolder, symbol Resistor_User:2k,0603
- D1: value NSR0530HT1G -> DFLS230L-7; footprint Diode_SMD:D_SOD-323_HandSoldering -> Diode_SMD:D_PowerDI-123; symbol Diode_User:NSR0530HT1G -> Diode_User:DFLS230L-7; MPN (none) -> DFLS230L-7; Manufacturer onsemi -> Diodes; SPN NSR0530HT1GOSCT-ND -> DFLS230LDICT-ND; Supplier Digi-Key -> DigiKey
- U1: value TPS563206 -> TPS564255; symbol Regulator_Switching:TPS563206 -> Regulator_Switching_User:TPS564255; MPN (none) -> TPS564255DRLR; Manufacturer (none) -> Texas Instruments; SPN (none) -> 296-TPS564257DRLRCT-ND; Supplier (none) -> DigiKey
Connections:
- net +Vout: now also J2.1 (Pin_1), J5.1 (Pin_1), R5.1
- net -Vout: now also D4.1 (K), J6.1 (Pin_1), J7.1 (Pin_1); no longer C6.2, R1.2, R2.1, U1.6 (FB)
- net GND: now also L1.1, L1.4, C11.2, C7.2, D2.1 (K), D3.1 (K), J2.2 (Pin_2), J4.2 (Pin_2), J5.2 (Pin_2), J6.2 (Pin_2), J7.2 (Pin_2), J8.2 (Pin_2), R6.1; no longer L1.2, L1.3
- net Vin: now also C11.1, C7.1, J4.1 (Pin_1), J8.1 (Pin_1), J9.1 (Pin_1), R4.1
- net at R3.2, U1.5 (EN): now also J9.2 (Pin_2)
- net at D1.2 (A): now also L1.3; no longer L1.4
- net at U1.2 (SW): now also L1.2; no longer L1.1
- new net: D3.2 (A), R5.2
- new net: D2.2 (A), R4.2
- new net: D4.2 (A), R6.2
- new net FB: C6.2, R1.2, R2.1, U1.6 (FB)
Other:
- note removed: "TPS564257"
- moved on the sheet: C1, C10, C2, C3, C4, C5, C6, C8, C9, D1, L1, R1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

Commit message: Finalize RevA
Parts:
- J9: value JST_B2B-PH-K-x -> Header_01x02_Wurth_61300211121; footprint Connector_JST:JST_PH_B2B-PH-K_1x02_P2.00mm_Vertical -> Connector_PinHeader_2.54mm:PinHeader_1x02_P2.54mm_Vertical; symbol Connector_User:JST_B2B-PH-K-x -> Connector_User:Pin_Header_01x02_Wurth_61300211121; MPN B2B-PH-K-S(LF)(SN) -> 61300211121; Manufacturer JST -> Wurth Electronics; Pretty Value (none) -> 01x02 Header; SPN 455-1262-ND -> 732-5315-ND
- R1: value 10k,0603 -> 22k,0603; symbol Resistor_User:10k,0603 -> Resistor_User:22k,0603; Resistance 10k -> 22k
- R2: value 10k,0603 -> 3k,0603; symbol Resistor_User:10k,0603 -> Resistor_User:3k,0603; Resistance 10k -> 3k
- R3: value 0R,0603 -> 10k,0603; symbol Resistor_User:0R,0603 -> Resistor_User:10k,0603; Resistance 0R -> 10k
Connections:
- net -Vout: now also J9.2 (Pin_2)
- net Vin: no longer J9.1 (Pin_1)
- net En: now reaches R3.2, U1.5 (EN)
- net En: now also J9.1 (Pin_1); no longer J9.2 (Pin_2)
Other:
- company: (none) -> fl0m0
- title: (none) -> Split Rail Supply
- moved on the sheet: J9
